File: pcb/badge-pcb.kicad_pcb (KiCad board)
At the start: 2 copper layers, 49 x 50 mm, 44 parts, among them IC1 LM4861M, J3 455-1750-1-ND, Q1 AO3415A, Q2 AO3415A, T1 MMUN2213LT1G, T3 JUMPER-SMT_2_NO_SILK, T5 JUMPER-SMT_2_NO_SILK

Commit message: Clean 3
Parts:
- R4: value 1K -> 4K7
Changed lines of the file:
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@@
 			)
 		)
-		(property "Value" "1K"
+		(property "Value" "4K7"
 			(at 1.5524 1.0011 90)
 			(unlocked yes)
@@
 		)
 		(property "Datasheet" ""
-			(at 0 0 270)
+			(at 0 0 90)
 			(layer "F.Fab")
 			(hide yes)
@@
 		)
 		(property "Description" ""
-			(at 0 0 270)
+			(at 0 0 90)
 			(layer "F.Fab")
 			(hide yes)
